Commit message: ROS2 with 3 motors

File: software/morphobot_ws/src/hybrid_robot_hardware/urdf/robot.urdf.xacro (robot description, xacro)
@@ -1,4 +1,4 @@
 <?xml version="1.0"?>
-<robot xmlns:xacro="http://www.ros.org/wiki/xacro" name="st3215_robot">
+<robot xmlns:xacro="http://www.ros.org/wiki/xacro" name="hybrid_robot_3servo">
   <!-- Base link -->
   <link name="base_link">
@@ -21,160 +21,125 @@
     </inertial>
   </link>
-  <!-- Macro for creating servo joints and links -->
-  <xacro:macro name="servo_joint" params="id parent">
-    <link name="servo_link_${id}">
-      <visual>
-        <geometry>
-          <cylinder radius="0.025" length="0.05"/>
-        </geometry>
-        <material name="blue">
-          <color rgba="0.2 0.2 0.8 1.0"/>
-        </material>
-      </visual>
-      <collision>
-        <geometry>
-          <cylinder radius="0.025" length="0.05"/>
-        </geometry>
-      </collision>
-      <inertial>
-        <mass value="0.1"/>
-        <inertia ixx="0.0001" ixy="0.0" ixz="0.0" iyy="0.0001" iyz="0.0" izz="0.0001"/>
-      </inertial>
-    </link>
-    <joint name="servo_joint_${id}" type="revolute">
-      <parent link="${parent}"/>
-      <child link="servo_link_${id}"/>
-      <origin xyz="0 0 0.05" rpy="0 0 0"/>
-      <axis xyz="0 0 1"/>
-      <limit lower="0" upper="6.28" effort="10.0" velocity="3.14"/>
-    </joint>
-  </xacro:macro>
-  <!-- Create 12 servo joints -->
-  <xacro:servo_joint id="1" parent="base_link"/>
-  <xacro:servo_joint id="2" parent="base_link"/>
-  <xacro:servo_joint id="3" parent="base_link"/>
-  <xacro:servo_joint id="4" parent="base_link"/>
-  <xacro:servo_joint id="5" parent="base_link"/>
-  <xacro:servo_joint id="6" parent="base_link"/>
-  <xacro:servo_joint id="7" parent="base_link"/>
-  <xacro:servo_joint id="8" parent="base_link"/>
-  <xacro:servo_joint id="9" parent="base_link"/>
-  <xacro:servo_joint id="10" parent="base_link"/>
-  <xacro:servo_joint id="11" parent="base_link"/>
-  <xacro:servo_joint id="12" parent="base_link"/>
+  <!-- Wheel link (driving servo) -->
+  <link name="wheel_fl_link">
+    <visual>
+      <geometry>
+        <cylinder radius="0.06" length="0.04"/>
+      </geometry>
+      <material name="blue">
+        <color rgba="0.2 0.2 0.8 1.0"/>
+      </material>
+    </visual>
+    <collision>
+      <geometry>
+        <cylinder radius="0.06" length="0.04"/>
+      </geometry>
+    </collision>
+    <inertial>
+      <mass value="0.2"/>
+      <inertia ixx="0.0001" ixy="0.0" ixz="0.0" iyy="0.0001" iyz="0.0" izz="0.0001"/>
+    </inertial>
+  </link>
+  <!-- Driving joint (continuous rotation) -->
+  <joint name="wheel_fl_joint" type="continuous">
+    <parent link="base_link"/>
+    <child link="wheel_fl_link"/>
+    <origin xyz="0.15 0.15 0" rpy="0 0 0"/>
+    <axis xyz="0 1 0"/>
+  </joint>
+  <!-- Pan mechanism link -->
+  <link name="pan_fl_link">
+    <visual>
+      <geometry>
+        <box size="0.05 0.05 0.08"/>
+      </geometry>
+      <material name="orange">
+        <color rgba="1.0 0.5 0.0 1.0"/>
+      </material>
+    </visual>
+    <collision>
+      <geometry>
+        <box size="0.05 0.05 0.08"/>
+      </geometry>
+    </collision>
+    <inertial>
+      <mass value="0.1"/>
+      <inertia ixx="0.00001" ixy="0.0" ixz="0.0" iyy="0.00001" iyz="0.0" izz="0.00001"/>
+    </inertial>
+  </link>
+  <!-- Pan joint (revolute - horizontal rotation) -->
+  <joint name="pan_fl_joint" type="revolute">
+    <parent link="base_link"/>
+    <child link="pan_fl_link"/>
+    <origin xyz="0.15 0.15 0.1" rpy="0 0 0"/>
+    <axis xyz="0 0 1"/>
+    <limit lower="-1.57" upper="1.57" effort="10.0" velocity="3.14"/>
+  </joint>
+  <!-- Tilt mechanism link -->
+  <link name="tilt_fl_link">
+    <visual>
+      <geometry>
+        <box size="0.08 0.03 0.03"/>
+      </geometry>
+      <material name="orange">
+        <color rgba="1.0 0.5 0.0 1.0"/>
+      </material>
+    </visual>
+    <collision>
+      <geometry>
+        <box size="0.08 0.03 0.03"/>
+      </geometry>
+    </collision>
+    <inertial>
+      <mass value="0.08"/>
+      <inertia ixx="0.00001" ixy="0.0" ixz="0.0" iyy="0.00001" iyz="0.0" izz="0.00001"/>
+    </inertial>
+  </link>
+  <!-- Tilt joint (revolute - vertical rotation) -->
+  <joint name="tilt_fl_joint" type="revolute">
+    <parent link="pan_fl_link"/>
+    <child link="tilt_fl_link"/>
+    <origin xyz="0 0 0.08" rpy="0 0 0"/>
+    <axis xyz="0 1 0"/>
+    <limit lower="-0.785" upper="0.785" effort="10.0" velocity="3.14"/>
+  </joint>
   <!-- ros2_control hardware interface -->
-  <ros2_control name="ST3215HardwareInterface" type="system">
+  <ros2_control name="ST3215Hardware" type="system">
     <hardware>
       <plugin>mock_components/GenericSystem</plugin>
-      <param name="mock_sensor_commands">false</param>
-      <param name="state_following">true</param>
+      <param name="port">/dev/ttyUSB0</param>
     </hardware>
-    <!-- Servo 1 -->
-    <joint name="servo_joint_1">
-      <command_interface name="position">
-        <param name="min">0</param>
-        <param name="max">6.28</param>
+    <!-- Driving joint (velocity control) -->
+    <joint name="wheel_fl_joint">
+      <command_interface name="velocity">
+        <param name="min">-10.0</param>
+        <param name="max">10.0</param>
       </command_interface>
       <state_interface name="position"/>
       <state_interface name="velocity"/>
+      <param name="servo_id">1</param>
+      <param name="mode">velocity</param>
     </joint>
-    <!-- Servo 2 -->
-    <joint name="servo_joint_2">
+    <!-- Pan joint (position control) -->
+    <joint name="pan_fl_joint">
       <command_interface name="position">
-        <param name="min">0</param>
-        <param name="max">6.28</param>
+        <param name="min">-1.57</param>
+        <param name="max">1.57</param>
       </command_interface>
       <state_interface name="position"/>
       <state_interface name="velocity"/>
+      <param name="servo_id">3</param>
+      <param name="mode">position</param>
     </joint>
-    <!-- Servo 3 -->
-    <joint name="servo_joint_3">
+    <!-- Tilt joint (position control) -->
+    <joint name="tilt_fl_joint">
       <command_interface name="position">
-        <param name="min">0</param>
-        <param name="max">6.28</param>
+        <param name="min">-0.785</param>
+        <param name="max">0.785</param>
       </command_interface>
       <state_interface name="position"/>
       <state_interface name="velocity"/>
-    </joint>
-    <!-- Servo 4 -->
-    <joint name="servo_joint_4">
-      <command_interface name="position">
-        <param name="min">0</param>
-        <param name="max">6.28</param>
-      </command_interface>
-      <state_interface name="position"/>
-      <state_interface name="velocity"/>
-    </joint>
-    <!-- Servo 5 -->
-    <joint name="servo_joint_5">
-      <command_interface name="position">
-        <param name="min">0</param>
-        <param name="max">6.28</param>
-      </command_interface>
-      <state_interface name="position"/>
-      <state_interface name="velocity"/>
-    </joint>
-    <!-- Servo 6 -->
-    <joint name="servo_joint_6">
-      <command_interface name="position">
-        <param name="min">0</param>
-        <param name="max">6.28</param>
-      </command_interface>
-      <state_interface name="position"/>
-      <state_interface name="velocity"/>
-    </joint>
-    <!-- Servo 7 -->
-    <joint name="servo_joint_7">
-      <command_interface name="position">
-        <param name="min">0</param>
-        <param name="max">6.28</param>
-      </command_interface>
-      <state_interface name="position"/>
-      <state_interface name="velocity"/>
-    </joint>
-    <!-- Servo 8 -->
-    <joint name="servo_joint_8">
-      <command_interface name="position">
-        <param name="min">0</param>
-        <param name="max">6.28</param>
-      </command_interface>
-      <state_interface name="position"/>
-      <state_interface name="velocity"/>
-    </joint>
-    <!-- Servo 9 -->
-    <joint name="servo_joint_9">
-      <command_interface name="position">
-        <param name="min">0</param>
-        <param name="max">6.28</param>
-      </command_interface>
-      <state_interface name="position"/>
-      <state_interface name="velocity"/>
-    </joint>
-    <!-- Servo 10 -->
-    <joint name="servo_joint_10">
-      <command_interface name="position">
-        <param name="min">0</param>
-        <param name="max">6.28</param>
-      </command_interface>
-      <state_interface name="position"/>
-      <state_interface name="velocity"/>
-    </joint>
-    <!-- Servo 11 -->
-    <joint name="servo_joint_11">
-      <command_interface name="position">
-        <param name="min">0</param>
-        <param name="max">6.28</param>
-      </command_interface>
-      <state_interface name="position"/>
-      <state_interface name="velocity"/>
-    </joint>
-    <!-- Servo 12 -->
-    <joint name="servo_joint_12">
-      <command_interface name="position">
-        <param name="min">0</param>
-        <param name="max">6.28</param>
-      </command_interface>
-      <state_interface name="position"/>
-      <state_interface name="velocity"/>
+      <param name="servo_id">4</param>
+      <param name="mode">position</param>
     </joint>
   </ros2_control>
