Commit message: Test with real mechanism

File: software/morphobot_ws/src/hybrid_robot_hardware/urdf/hybrid_robot.urdf.xacro (robot description, xacro)
@@ -3,6 +3,6 @@
   <!-- Define servo joint names and IDs -->
   <xacro:property name="servo_1_id" value="1" />
+  <xacro:property name="servo_2_id" value="2" />
   <xacro:property name="servo_3_id" value="3" />
-  <xacro:property name="servo_4_id" value="4" />
   <!-- Base link -->
   <link name="base_link">
@@ -34,4 +34,22 @@
     <limit lower="-3.14" upper="3.14" effort="10" velocity="5"/>
   </joint>
+  <!-- Servo 2 link and joint -->
+  <link name="servo_link_2">
+    <visual>
+      <geometry>
+        <cylinder radius="0.02" length="0.05"/>
+      </geometry>
+      <material name="gray">
+        <color rgba="0.5 0.5 0.5 1"/>
+      </material>
+    </visual>
+  </link>
+  <joint name="servo_joint_2" type="revolute">
+    <parent link="base_link"/>
+    <child link="servo_link_2"/>
+    <origin xyz="0 0.05 0" rpy="0 0 0"/>
+    <axis xyz="0 0 1"/>
+    <limit lower="-3.14" upper="3.14" effort="10" velocity="5"/>
+  </joint>
   <!-- Servo 3 link and joint -->
   <link name="servo_link_3">
@@ -48,22 +66,4 @@
     <parent link="base_link"/>
     <child link="servo_link_3"/>
-    <origin xyz="0 0.05 0" rpy="0 0 0"/>
-    <axis xyz="0 0 1"/>
-    <limit lower="-3.14" upper="3.14" effort="10" velocity="5"/>
-  </joint>
-  <!-- Servo 4 link and joint -->
-  <link name="servo_link_4">
-    <visual>
-      <geometry>
-        <cylinder radius="0.02" length="0.05"/>
-      </geometry>
-      <material name="gray">
-        <color rgba="0.5 0.5 0.5 1"/>
-      </material>
-    </visual>
-  </link>
-  <joint name="servo_joint_4" type="revolute">
-    <parent link="base_link"/>
-    <child link="servo_link_4"/>
     <origin xyz="-0.05 0 0" rpy="0 0 0"/>
     <axis xyz="0 0 1"/>
@@ -75,5 +75,5 @@
       <plugin>hybrid_robot_hardware/ST3215HardwareInterface</plugin>
       <param name="serial_port">/dev/ttyUSB0</param>
-      <param name="servo_ids">1,3,4</param>
+      <param name="servo_ids">1,2,3</param>
     </hardware>
     <joint name="servo_joint_1">
@@ -82,4 +82,18 @@
         <param name="max">3.14</param>
       </command_interface>
+      <state_interface name="position"/>
+      <state_interface name="velocity"/>
+      <state_interface name="effort"/>
+    </joint>
+    <joint name="servo_joint_2">
+      <command_interface name="position">
+        <param name="min">-3.14</param>
+        <param name="max">3.14</param>
+      </command_interface>
+      <state_interface name="position"/>
+      <state_interface name="velocity"/>
+      <state_interface name="effort"/>
+    </joint>
+    <joint name="servo_joint_3">
       <command_interface name="velocity">
         <param name="min">-5.0</param>
@@ -90,22 +104,4 @@
       <state_interface name="effort"/>
     </joint>
-    <joint name="servo_joint_3">
-      <command_interface name="position">
-        <param name="min">-3.14</param>
-        <param name="max">3.14</param>
-      </command_interface>
-      <state_interface name="position"/>
-      <state_interface name="velocity"/>
-      <state_interface name="effort"/>
-    </joint>
-    <joint name="servo_joint_4">
-      <command_interface name="position">
-        <param name="min">-3.14</param>
-        <param name="max">3.14</param>
-      </command_interface>
-      <state_interface name="position"/>
-      <state_interface name="velocity"/>
-      <state_interface name="effort"/>
-    </joint>
   </ros2_control>
 </robot>
