Commit message: add vision system

File: software/morphobot_ws/src/morphobot_urdf/urdf/hybrid_robot.urdf.xacro (robot description, xacro)
@@ -51,5 +51,5 @@
     <child link="servo_bracket_FR" />
     <axis xyz="1 0 0" />
-    <limit lower="-3.14" upper="3.14" effort="10.0" velocity="5.0" />
+    <limit lower="-3.14" upper="3.14" effort="50.0" velocity="5.0" />
   </joint>
   <link name="append_FR">
@@ -167,5 +167,5 @@
     <child link="servo_bracket_FL" />
     <axis xyz="1 0 0" />
-    <limit lower="-3.14" upper="3.14" effort="10.0" velocity="5.0" />
+    <limit lower="-3.14" upper="3.14" effort="50.0" velocity="5.0" />
   </joint>
   <link name="append_FL">
@@ -488,129 +488,73 @@
     <limit effort="10.0" velocity="5.0" />
   </joint>
-<ros2_control name="ST3215HardwareSystem" type="system">
-    <hardware>
-      <xacro:if value="$(arg sim_mode)">
-        <plugin>gz_ros2_control/GazeboSimSystem</plugin>
-      </xacro:if>
-      <xacro:unless value="$(arg sim_mode)">
-        <plugin>ugv_motor_driver/ST3215HardwareInterface</plugin>
-        <param name="serial_port">/dev/ttyUSB0</param>
-        <param name="servo_ids">1,2,3,4,5,6,7,8,9,10,11,12</param>
-      </xacro:unless>
-    </hardware>
-    <joint name="hip_FL">
-      <command_interface name="position">
-        <param name="min">-3.14</param>
-        <param name="max">3.14</param>
-      </command_interface>
-      <state_interface name="position" />
-      <state_interface name="velocity" />
-      <state_interface name="effort" />
-    </joint>
-    <joint name="ankle_FL">
-      <command_interface name="position">
-        <param name="min">-3.14</param>
-        <param name="max">3.14</param>
-      </command_interface>
-      <state_interface name="position" />
-      <state_interface name="velocity" />
-      <state_interface name="effort" />
-    </joint>
-    <joint name="drive_FL">
-      <command_interface name="velocity">
-        <param name="min">-255</param>
-        <param name="max">255</param>
-      </command_interface>
-      <state_interface name="position" />
-      <state_interface name="velocity" />
-      <state_interface name="effort" />
-    </joint>
-    <joint name="hip_BL">
-      <command_interface name="position">
-        <param name="min">-3.14</param>
-        <param name="max">3.14</param>
-      </command_interface>
-      <state_interface name="position" />
-      <state_interface name="velocity" />
-      <state_interface name="effort" />
-    </joint>
-    <joint name="ankle_BL">
-      <command_interface name="position">
-        <param name="min">-3.14</param>
-        <param name="max">3.14</param>
-      </command_interface>
-      <state_interface name="position" />
-      <state_interface name="velocity" />
-      <state_interface name="effort" />
-    </joint>
-    <joint name="drive_BL">
-      <command_interface name="velocity">
-        <param name="min">-255</param>
-        <param name="max">255</param>
-      </command_interface>
-      <state_interface name="position" />
-      <state_interface name="velocity" />
-      <state_interface name="effort" />
-    </joint>
-    <joint name="hip_FR">
-      <command_interface name="position">
-        <param name="min">-3.14</param>
-        <param name="max">3.14</param>
-      </command_interface>
-      <state_interface name="position" />
-      <state_interface name="velocity" />
-      <state_interface name="effort" />
-    </joint>
-    <joint name="ankle_FR">
-      <command_interface name="position">
-        <param name="min">-3.14</param>
-        <param name="max">3.14</param>
-      </command_interface>
-      <state_interface name="position" />
-      <state_interface name="velocity" />
-      <state_interface name="effort" />
-    </joint>
-    <joint name="drive_FR">
-      <command_interface name="velocity">
-        <param name="min">-255</param>
-        <param name="max">255</param>
-      </command_interface>
-      <state_interface name="position" />
-      <state_interface name="velocity" />
-      <state_interface name="effort" />
-    </joint>
-    <joint name="hip_BR">
-      <command_interface name="position">
-        <param name="min">-3.14</param>
-        <param name="max">3.14</param>
-      </command_interface>
-      <state_interface name="position" />
-      <state_interface name="velocity" />
-      <state_interface name="effort" />
-    </joint>
-    <joint name="ankle_BR">
-      <command_interface name="position">
-        <param name="min">-3.14</param>
-        <param name="max">3.14</param>
-      </command_interface>
-      <state_interface name="position" />
-      <state_interface name="velocity" />
-      <state_interface name="effort" />
-    </joint>
-    <joint name="drive_BR">
-      <command_interface name="velocity">
-        <param name="min">-255</param>
-        <param name="max">255</param>
-      </command_interface>
-      <state_interface name="position" />
-      <state_interface name="velocity" />
-      <state_interface name="effort" />
-    </joint>
-  </ros2_control>
+<ros2_control name="GazeboSystem" type="system">
+  <hardware>
+    <plugin>ign_ros2_control/IgnitionSystem</plugin>
+  </hardware>
+  <!-- Hip joints -->
+  <joint name="hip_FL">
+    <command_interface name="position"/>
+    <state_interface name="position"/>
+    <state_interface name="velocity"/>
+  </joint>
+  <joint name="hip_FR">
+    <command_interface name="position"/>
+    <state_interface name="position"/>
+    <state_interface name="velocity"/>
+  </joint>
+  <joint name="hip_BL">
+    <command_interface name="position"/>
+    <state_interface name="position"/>
+    <state_interface name="velocity"/>
+  </joint>
+  <joint name="hip_BR">
+    <command_interface name="position"/>
+    <state_interface name="position"/>
+    <state_interface name="velocity"/>
+  </joint>
+  <!-- Ankle joints -->
+  <joint name="ankle_FL">
+    <command_interface name="position"/>
+    <state_interface name="position"/>
+    <state_interface name="velocity"/>
+  </joint>
+  <joint name="ankle_FR">
+    <command_interface name="position"/>
+    <state_interface name="position"/>
+    <state_interface name="velocity"/>
+  </joint>
+  <joint name="ankle_BL">
+    <command_interface name="position"/>
+    <state_interface name="position"/>
+    <state_interface name="velocity"/>
+  </joint>
+  <joint name="ankle_BR">
+    <command_interface name="position"/>
+    <state_interface name="position"/>
+    <state_interface name="velocity"/>
+  </joint>
+  <!-- Drive wheels -->
+  <joint name="drive_FL">
+    <command_interface name="velocity"/>
+    <state_interface name="velocity"/>
+  </joint>
+  <joint name="drive_FR">
+    <command_interface name="velocity"/>
+    <state_interface name="velocity"/>
+  </joint>
+  <joint name="drive_BL">
+    <command_interface name="velocity"/>
+    <state_interface name="velocity"/>
+  </joint>
+  <joint name="drive_BR">
+    <command_interface name="velocity"/>
+    <state_interface name="velocity"/>
+  </joint>
+</ros2_control>
   <gazebo>
     <plugin
-      filename="libgz_ros2_control-system.so"
-      name="gz_ros2_control::GazeboSimROS2ControlPlugin">
-      <parameters>$(find ugv_motor_driver)/config/controllers.yaml</parameters>
+      filename="libign_ros2_control-system.so"
+      name="ign_ros2_control::IgnitionROS2ControlPlugin">
+      <parameters>$(find morphobot_urdf)/config/sim_controllers.yaml</parameters>
     </plugin>
   </gazebo>
